File: E1201/E1201.kicad_pcb (KiCad board)
At the start: 2 copper layers, 83.8 x 43.1 mm, 52 parts, among them J1 Screw_Terminal_01x02, J2 Screw_Terminal_01x04, J3 Conn_01x04_Socket, J4 Conn_01x06_Socket, J6 Conn_02x08_Odd_Even, J7 Conn_01x18, J9 QWIIC, Q1 MMBF170, Q2 MMBF170, Q3 MMBF170, SW1 SW_Push, U1 TXU0304PW, U2 TXU0202DCU, U3 TCA9517ADGK, U4 TPS61222DCK, U5 PIC16F18154-xSTX, U6 LM2776

Commit message: save point
Parts:
- added J8: ICSP, Connector:Tag-Connect_TC2030-IDC-NL_2x03_P1.27mm_Vertical, F.Cu at (177.1, 79.0)
- J6: footprint Connector_PinSocket_2.54mm:PinSocket_2x08_P2.54mm_Vertical -> Connector_PinHeader_2.54mm:PinHeader_2x08_P2.54mm_Vertical; moved to B.Cu
- J7: moved to B.Cu
- moved SW1 8.47 mm to (170.0, 84.6), turned to 180 degrees
- moved R8 1.36 mm to (174.6, 83.0), turned to -90 degrees
- turned J6 to 0 degrees
- turned J7 to 90 degrees
Routing:
- net /PROG_RST: track 17.2 -> 0.00 mm, vias 2 -> 0
- net VIN: track 76.3 -> 71.8 mm
- net /LCD_{BIAS}: track 26.5 -> 30.7 mm, vias 0 -> 1
- net +5V: track 219.0 -> 217.6 mm
