File: E1201/E1201.kicad_sch (KiCad schematic)
At the start: 53 parts, among them J1 Screw_Terminal_01x02, J2 Screw_Terminal_01x04, J3 Conn_01x04_Socket, J4 Conn_01x06_Socket, J6 Conn_02x08_Odd_Even, J7 Conn_01x18, J8 ICSP, J9 QWIIC, Q1 MMBF170, Q2 MMBF170, Q3 MMBF170, SW1 SW_Push, U1 TXU0304PW, U2 TXU0202DCU, U3 TCA9517ADGK, U4 TPS61222DCK, U5 PIC16F18154-xSTX, U6 LM2776

Commit message: save point
Parts:
- J6: footprint Connector_PinSocket_2.54mm:PinSocket_2x08_P2.54mm_Vertical -> Connector_PinHeader_2.54mm:PinHeader_2x08_P2.54mm_Vertical
Changed lines of the file:
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@@
 			)
 		)
-		(property "Footprint" "Connector_PinSocket_2.54mm:PinSocket_2x08_P2.54mm_Vertical"
+		(property "Footprint" "Connector_PinHeader_2.54mm:PinHeader_2x08_P2.54mm_Vertical"
 			(at 381 106.68 0)
 			(hide yes)
