File: E1201/E1201.kicad_sch (KiCad schematic)
At the start: 53 parts, among them J1 Screw_Terminal_01x02, J2 Screw_Terminal_01x04, J3 Conn_01x04_Socket, J4 Conn_01x06_Socket, J6 Conn_02x08_Odd_Even, J7 Conn_01x18, J8 ICSP, J9 QWIIC, Q1 MMBF170, Q2 MMBF170, Q3 MMBF170, SW1 SW_Push, U1 TXU0304PW, U2 TXU0202DCU, U3 TCA9517ADGK, U4 TPS61222DCK, U5 PIC16F18154-xSTX, U6 LM2776

Commit message: PCB Commit, this is what I used to order
Parts:
- removed J2: Screw_Terminal_01x04, Connector_PinSocket_2.54mm:PinSocket_1x04_P2.54mm_Horizontal, symbol Connector:Screw_Terminal_01x04
- removed JP1: Jumper_3_Open, Jumper:SolderJumper-3_P2.0mm_Open_TrianglePad1.0x1.5mm_NumberLabels, symbol Jumper:Jumper_3_Open
- removed U5: PIC16F18154-xSTX, Package_DFN_QFN:QFN-28-1EP_4x4mm_P0.4mm_EP2.4x2.4mm, symbol MCU_Microchip_PIC16:PIC16F18154-xSTX
- added J2: Conn_01x04_Socket, Connector_PinSocket_2.54mm:PinSocket_1x04_P2.54mm_Vertical, symbol Connector:Conn_01x04_Socket
- added TP1, TP2: TestPoint, TestPoint:TestPoint_Pad_1.5x1.5mm, symbol Connector:TestPoint
- added U5: PIC16F18154-xSS, Package_SO:SSOP-28_5.3x10.2mm_P0.65mm, symbol MCU_Microchip_PIC16:PIC16F18154-xSS
- C3: renamed from C2; value C -> 10uF
- C7: renamed from C3; value C -> 10uF
- J1: footprint Connector_PinSocket_2.54mm:PinSocket_1x02_P2.54mm_Horizontal -> Connector_PinSocket_2.54mm:PinSocket_1x02_P2.54mm_Vertical
- J3: footprint Connector_PinSocket_2.54mm:PinSocket_1x04_P2.54mm_Horizontal -> Connector_PinSocket_2.54mm:PinSocket_1x04_P2.54mm_Vertical
- J4: footprint Connector_PinSocket_2.54mm:PinSocket_1x06_P2.54mm_Horizontal -> Connector_PinSocket_2.54mm:PinSocket_1x06_P2.54mm_Vertical
- J6: renamed from J8; footprint Connector_PinSocket_2.54mm:PinSocket_1x06_P2.54mm_Vertical -> Connector:Tag-Connect_TC2030-IDC-NL_2x03_P1.27mm_Vertical
- L1: value L -> 4.7uH; footprint Inductor_SMD:L_1206_3216Metric_Pad1.22x1.90mm_HandSolder -> Inductor_SMD:L_1210_3225Metric; Part Number (none) -> CBC3225T4R7MR
- R6: value 10k -> 20k
- R7: value 10k -> 180k
- renumbered C6 to C10, C7 to C2, C9 to C4, C8 to C5, C10 to C6, C4 to C8, C5 to C9, J9 to J5, J6 to J7, J7 to J8, JP2 to JP1, R15 to R12, R16 to R13, R17 to R14, R9 to R8, R8 to R9
Connections:
- net +5V: now also TP1.1, U5.20 (VDD)
- net GND: now also J2.3 (Pin_3), TP2.1, U5.19 (VSS), U5.8 (VSS)
- net LCD_{BL_{1}}_EN: now also U5.23 (RB2)
- net LCD_{BL_{2}}_EN: now also U5.22 (RB1)
- net LCD_{BL_{3}}_EN: now also U5.21 (RB0)
- net LCD_{D0}: now also U5.2 (RA0)
- net LCD_{D1}: now also U5.3 (RA1)
- net LCD_{D2}: now also U5.4 (RA2)
- net LCD_{D3}: now also U5.5 (RA3)
- net LCD_{D4}: now also U5.6 (RA4)
- net LCD_{D5}: now also U5.7 (RA5)
- net LCD_{D6}: now also U5.9 (RA7)
- net LCD_{D7}: now also U5.10 (RA6)
- net LCD_{EN}: now also U5.24 (RB3)
- net LCD_{RS}: now also U5.26 (RB5)
- net LCD_{RW}: now also U5.25 (RB4)
- net MCU_I2C_SCL: now also U5.14 (RC3)
- net MCU_I2C_SDA: now also U5.15 (RC4)
- net MCU_SPI_CLK: now also U5.13 (RC2)
- net MCU_SPI_MISO: now also U5.16 (RC5)
- net MCU_SPI_MOSI: now also U5.12 (RC1)
- net MCU_SPI_~{CS}: now also U5.11 (RC0)
- net MCU_UART_RX: now also U5.18 (RC7)
- net MCU_UART_TX: now also U5.17 (RC6)
- net PROG_CLK: now also U5.27 (RB6/ICSPCLK)
- net PROG_DAT: now also U5.28 (RB7/ICSPDAT)
- net UART_RX: now also J2.2 (Pin_2)
- net UART_TX: now also J2.1 (Pin_1)
- net VIN: now also J2.4 (Pin_4)
- net VIN-P: now also C3.2, L1.1, U4.1 (VIN), U4.6 (EN)
- net PROG_RST renamed PROG_VPP
- net PROG_VPP: now also U5.1 (RE3/~{MCLR}/VPP)
Other:
- note added: "5V Supply"
- note added: "Backlight Drivers"
- note added: "External Pullups"
- note added: "Input Conditioning"
- note added: "Inputs"
- note added: "LCD Bias Gen"
- note added: "LCDs"
- note added: "Microcontroller"
- note added: "Misc"
- note added: "Programming"
- note added: "Protection"
- note added: "Pull-Ups"
- moved on the sheet: C1, C3, C7, D1, D2, D3, F1, FB1, H1, L1, R10, R11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
